File: mchck.kicad_pcb (KiCad board)
At the start: 2 copper layers, 45.7 x 19.1 mm, 33 parts, among them J3 MICRO_USB, K1 CONN_MICROSD, P2 CONN_1, P3 UPPER_PINS, P4 LOWER_PINS, P6 JTAG, U1 MK20LF, U2 MCP1703_SOT23, X1 8MHz, Y1 32.768kHz

Commit message: Final tidy up for V2.
Parts:
- removed P2: CONN_1, RMC_pcb_header:pin_header_2.54mm_1x1
- X1: footprint RMC:XTAL-SM-TXC-7A -> Crystals:Crystal_SMD_0603_4Pads
- moved C9 5.34 mm to (54.0, 55.2), turned to 270 degrees
- moved C13 3.81 mm to (62.9, 55.2), turned to 90 degrees
- moved X1 1.65 mm to (58.4, 54.6)
- moved FB1 0.90 mm to (55.9, 51.2)
- moved Y1 0.52 mm to (49.0, 55.8)
- turned G1 to 270 degrees
Connections:
- net A18 renamed /MCU/A18
- C13 pad 1: A19 -> /MCU/A19
- P3 pad 1: VRAW -> VBUS
- P4 pad 2: Net-(P4-Pad2) -> VRAW
- P4 pad 3: ADC0+ -> VBAT
- P4 pad 4: ADC0- -> ADC0+
- P4 pad 5: VREFH -> ADC0-
- P4 pad 6: VBAT -> VREFH
- U1 pad 25: A19 -> /MCU/A19
- X1 pad 2: A19 -> Net-(X1-Pad2)
Routing:
- net VRAW: track 40.9 -> 22.7 mm
- net VBAT: track 6.59 -> 16.4 mm
- net A19: track 5.25 -> 0.00 mm, vias 1 -> 0
- net /MCU/A19: track 0.00 -> 4.33 mm, vias 0 -> 1
- net VBUS: track 13.6 -> 17.9 mm
- net ADC0+: track 14.6 -> 12.7 mm
- net /MCU/A18: track 6.00 -> 7.28 mm
- net Net-(U1-Pad14): track 2.89 -> 4.02 mm
- net Net-(U1-Pad15): track 3.31 -> 4.31 mm
Other:
- board text added: "VRH"
- board text removed: "A18"
- board text removed: "A19"
- board text removed: "CK"
- board text removed: "IO"
