File: mchck.sch (KiCad schematic (older format))
At the start: 6 parts, among them P1 RIGHT_PINS, P2 DEBUG, P3 UPPER_PINS, P4 LOWER_PINS

Commit message: Mash up of MCHCK with TinyK20-like pinout
Parts:
- removed H1: MOUNTHOLE, mounthole_3mm, symbol MOUNTHOLE
- removed P1: RIGHT_PINS, SparkFun-1X06_LOCK, symbol CONN_6
- removed P2: DEBUG, SparkFun-1X04_LOCK, symbol CONN_4
- added M1: PCB_GREEN_RMC, ~, symbol PCB_GREEN_RMC
- added P2: CONN_1, symbol CONN_1
- P3, P4: symbol CONN_14 -> CONN_18
Connections:
- net labels added: A0, A1, A18, A19, A2, A3, A4, ADC0+, ADC0-, B0, B1, B16, B17, B2, B3, C0, C1, C2, C3, C4, C5, C6, C7, D0, D1, D2, D3, D4, D5, D6, D7, RST, VBAT, VBUS, VRAW, VREFH, VREFL
- wire segments 51 -> 37
Other:
- note added: "BC-HCK version 1 \nBob Cousins Jan 2015"
- note added: "TODO\n\nDIP 32?\n- VREF pin\n- move VRAW"

Commit message: Fix up libs and footprints for Kicad v4; remove several unused libs
Parts:
- removed M1: PCB_GREEN_RMC, ~, symbol PCB_GREEN_RMC
- removed P3: UPPER_PINS, SparkFun-1X14_LOCK, symbol CONN_18
- added P3: UPPER_PINS, RMC_pcb_header:pin_header_2.54mm_1x18, symbol CONN_01X18
- G1: footprint OHW-LOGO-6mm -> mchck:OHW-LOGO-6mm
- P2: footprint (none) -> RMC_pcb_header:pin_header_2.54mm_1x1; symbol CONN_1 -> CONN_01X01
- P4: footprint SparkFun-1X14_LOCK -> RMC_pcb_header:pin_header_2.54mm_1x18; symbol CONN_18 -> CONN_01X18
Connections:
- net labels added: GND
- net labels removed: VSS
Changed lines of the file:
@@
 EESchema Schematic File Version 2
 LIBS:mchck-rescue
-LIBS:usb
 LIBS:power
 LIBS:device
@@
 LIBS:74xx
 LIBS:cmos4000
-LIBS:adc-dac
-LIBS:memory
-LIBS:xilinx
-LIBS:microcontrollers
-LIBS:dsp
-LIBS:microchip
-LIBS:analog_switches
-LIBS:motorola
-LIBS:texas
-LIBS:intel
-LIBS:audio
-LIBS:interface
-LIBS:digital-audio
-LIBS:philips
-LIBS:display
-LIBS:cypress
-LIBS:siliconi
-LIBS:opto
-LIBS:atmel
-LIBS:contrib
-LIBS:valves
-LIBS:microsd
-LIBS:conn_16
-LIBS:conn_15
-LIBS:conn_18
-LIBS:mcp73831
 LIBS:SparkFun
 LIBS:tac_switchsmd_evqp2
-LIBS:cn3063
-LIBS:mic5205
-LIBS:NUC120_QFN48
-LIBS:mcp1702
-LIBS:multireg
-LIBS:inductor_select
 LIBS:logo
 LIBS:MK20LF
-LIBS:mounthole
-LIBS:vssa
-LIBS:vdda
 LIBS:RMC
 LIBS:opendous
@@
 $EndDescr
 $Comp
-L CONN_18 P4
+L CONN_01X18 P4
 U 1 1 4E446864
-P 4350 6200
-F 0 "P4" V 4300 6200 60  0000 C CNN
-F 1 "LOWER_PINS" V 4400 6200 60  0000 C CNN
-F 2 "SparkFun-1X14_LOCK" V 4350 6200 60  0001 C CNN
-F 3 "" H 4350 6200 60  0001 C CNN
-F 4 "never" V 4350 6200 60  0001 C CNN "populate"
-	1    4350 6200
+P 4350 6050
+F 0 "P4" H 4350 7000 50  0000 C CNN
+F 1 "LOWER_PINS" V 4450 6050 50  0000 C CNN
+F 2 "RMC_pcb_header:pin_header_2.54mm_1x18" H 4350 6050 50  0001 C CNN
+F 3 "" H 4350 6050 50  0000 C CNN
+F 4 "never" V 4350 6050 60  0001 C CNN "populate"
+	1    4350 6050
 	0    -1   1    0
-$EndComp
-$Comp
-L CONN_18 P3
-U 1 1 4E446858
-P 4350 3200
-F 0 "P3" V 4300 3200 60  0000 C CNN
-F 1 "UPPER_PINS" V 4400 3200 60  0000 C CNN
-F 2 "SparkFun-1X14_LOCK" V 4350 3200 60  0001 C CNN
-F 3 "" H 4350 3200 60  0001 C CNN
-F 4 "never" V 4350 3200 60  0001 C CNN "populate"
-	1    4350 3200
-	0    -1   -1   0
 $EndComp
 $Comp
@@
 F 0 "G1" H 10300 800 60  0000 C CNN
 F 1 "OHW LOGO" H 10300 550 60  0000 C CNN
-F 2 "OHW-LOGO-6mm" H 10300 650 60  0001 C CNN
+F 2 "mchck:OHW-LOGO-6mm" H 10300 650 60  0001 C CNN
 F 3 "" H 10300 800 60  0001 C CNN
 F 4 "never" H 10300 800 60  0001 C CNN "populate"
@@
 Wire Wire Line
 	4700 5850 4700 5600
-$Comp
-L PCB_GREEN_RMC M1
-U 1 1 54C3842E
-P 9400 1000
-F 0 "M1" H 9400 1150 60  0000 C CNN
-F 1 "PCB_GREEN_RMC" H 9400 900 60  0000 C CNN
-F 2 "~" H 9400 1000 60  0000 C CNN
-F 3 "~" H 9400 1000 60  0000 C CNN
-	1    9400 1000
-	1    0    0    -1
-$EndComp
 $Sheet
 S 7350 4800 1050 600
@@
 F1 "mcu.sch" 60
 $EndSheet
-Text Notes 650  1100 0    100  ~ 0
+Text Notes 900  1800 0    100  ~ 0
 TODO\n\nDIP 32?\n- VREF pin\n- move VRAW
-Text Notes 7200 6750 0    80   ~ 0
+Text Notes 7050 6850 0    80   ~ 0
 BC-HCK version 1 \nBob Cousins Jan 2015
 Wire Wire Line
@@
 RST
 $Comp
-L VSS #PWR01
-U 1 1 56558BB5
-P 3350 5200
-F 0 "#PWR01" H 3350 5200 30  0001 C CNN
-F 1 "VSS" H 3350 5130 30  0000 C CNN
-F 2 "" H 3350 5200 60  0000 C CNN
-F 3 "" H 3350 5200 60  0000 C CNN
-	1    3350 5200
-	1    0    0    -1
-$EndComp
-$Comp
-L VDD #PWR02
+L VDD #PWR01
 U 1 1 56558A41
 P 5200 4200
-F 0 "#PWR02" H 5200 4300 30  0001 C CNN
+F 0 "#PWR01" H 5200 4300 30  0001 C CNN
 F 1 "VDD" H 5200 4310 30  0000 C CNN
 F 2 "" H 5200 4200 60  0000 C CNN
@@
 VREFH
 $Comp
-L CONN_1 P2
+L CONN_01X01 P2
 U 1 1 56564A1C
-P 2900 3300
-F 0 "P2" H 2980 3300 40  0000 L CNN
-F 1 "CONN_1" H 2900 3355 30  0001 C CNN
-F 2 "" H 2900 3300 60  0000 C CNN
-F 3 "" H 2900 3300 60  0000 C CNN
-	1    2900 3300
+P 2950 3350
+F 0 "P2" H 3030 3350 40  0000 L CNN
+F 1 "CONN_1" H 2950 3405 30  0001 C CNN
+F 2 "RMC_pcb_header:pin_header_2.54mm_1x1" H 2950 3200 60  0001 C CNN
+F 3 "" H 2950 3350 60  0000 C CNN
+	1    2950 3350
 	0    -1   -1   0
 $EndComp
 Text GLabel 2550 5800 1    40   Input ~ 0
 VREFL
-Text GLabel 2900 3450 3    40   Input ~ 0
+Text GLabel 2950 3550 3    40   Input ~ 0
 VBUS
 Wire Wire Line
@@
 Wire Wire Line
 	5200 5850 5200 5600
+$Comp
+L GND #PWR02
+U 1 1 566F8983
+P 3350 5200
+F 0 "#PWR02" H 3350 4950 50  0001 C CNN
+F 1 "GND" H 3350 5050 50  0000 C CNN
+F 2 "" H 3350 5200 50  0000 C CNN
+F 3 "" H 3350 5200 50  0000 C CNN
+	1    3350 5200
+	1    0    0    -1
+$EndComp
+$Comp
+L CONN_01X18 P3
+U 1 1 568284A5
+P 4350 3350
+F 0 "P3" H 4350 4300 50  0000 C CNN
+F 1 "UPPER_PINS" V 4450 3350 50  0000 C CNN
+F 2 "RMC_pcb_header:pin_header_2.54mm_1x18" H 4350 3350 50  0001 C CNN
+F 3 "" H 4350 3350 50  0000 C CNN
+	1    4350 3350
+	0    -1   -1   0
+$EndComp
 $EndSCHEMATC

Commit message: Tidy up some texts; add doc files
Other:
- note removed: "BC-HCK version 1 \nBob Cousins Jan 2015"
Changed lines of the file:
@@
 EESchema Schematic File Version 2
-LIBS:mchck-rescue
 LIBS:power
 LIBS:device
@@
 encoding utf-8
 Sheet 1 4
-Title "MC HCK microcontroller board"
-Date "29 nov 2015"
-Rev "R5-rc3"
-Comp "(c) 2011,2012,2013 Simon Schubert"
-Comment1 "CERN OHL v.1.1 or later"
-Comment2 ""
+Title "BC HCK K20 "
+Date "2016-01-01"
+Rev "v2"
+Comp "License: CERN OHL v.1.1 or later"
+Comment1 "Copyright Bob Cousins 2016"
+Comment2 "Derived from MC HCK microcontroller board by Simon Schubert"
 Comment3 ""
 Comment4 ""
@@
 Text Notes 900  1800 0    100  ~ 0
 TODO\n\nDIP 32?\n- VREF pin\n- move VRAW
-Text Notes 7050 6850 0    80   ~ 0
-BC-HCK version 1 \nBob Cousins Jan 2015
 Wire Wire Line
 	4900 3900 4900 3550

Commit message: Final tidy up for V2.
Parts:
- removed P2: CONN_1, RMC_pcb_header:pin_header_2.54mm_1x1, symbol CONN_01X01
Connections:
- net labels removed: A18, A19, VREFL
- wire segments 37 -> 38
Other:
- note removed: "TODO\n\nDIP 32?\n- VREF pin\n- move VRAW"
Changed lines of the file:
@@
 LIBS:RMC
 LIBS:opendous
+LIBS:multireg
+LIBS:inductor_select
 LIBS:mchck-cache
 EELAYER 25 0
@@
 F1 "mcu.sch" 60
 $EndSheet
-Text Notes 900  1800 0    100  ~ 0
-TODO\n\nDIP 32?\n- VREF pin\n- move VRAW
 Wire Wire Line
 	4900 3900 4900 3550
@@
 Text GLabel 4900 3900 3    40   3State ~ 0
 C2
-Text GLabel 3500 3900 3    40   Output ~ 0
+Text GLabel 3600 5600 1    40   Output ~ 0
 VRAW
 Wire Wire Line
@@
 Wire Wire Line
 	4900 5600 4900 5850
+Text GLabel 3800 5600 1    40   Output ~ 0
+ADC0+
+Text GLabel 3900 5600 1    40   Output ~ 0
+ADC0-
 Text GLabel 3700 5600 1    40   Output ~ 0
-ADC0+
-Text GLabel 3800 5600 1    40   Output ~ 0
-ADC0-
-Text GLabel 4000 5600 1    40   Output ~ 0
 VBAT
 Text GLabel 4100 5600 1    40   3State ~ 0
@@
 Text GLabel 4500 5600 1    40   3State ~ 0
 A4
-Text GLabel 5750 5500 1    40   3State ~ 0
-A18
-Text GLabel 5850 5500 1    40   3State ~ 0
-A19
 Text GLabel 4600 5600 1    40   3State ~ 0
 B0
@@
 	-1   0    0    1
 $EndComp
-Text GLabel 3900 5600 1    40   Input ~ 0
+Text GLabel 4000 5600 1    40   Input ~ 0
 VREFH
-$Comp
-L CONN_01X01 P2
-U 1 1 56564A1C
-P 2950 3350
-F 0 "P2" H 3030 3350 40  0000 L CNN
-F 1 "CONN_1" H 2950 3405 30  0001 C CNN
-F 2 "RMC_pcb_header:pin_header_2.54mm_1x1" H 2950 3200 60  0001 C CNN
-F 3 "" H 2950 3350 60  0000 C CNN
-	1    2950 3350
-	0    -1   -1   0
-$EndComp
-Text GLabel 2550 5800 1    40   Input ~ 0
-VREFL
-Text GLabel 2950 3550 3    40   Input ~ 0
+Text GLabel 3500 3900 3    40   Input ~ 0
 VBUS
 Wire Wire Line
@@
 	0    -1   -1   0
 $EndComp
+Wire Wire Line
+	3600 5600 3600 5850
 $EndSCHEMATC
