File: mcu.sch (KiCad schematic (older format))
At the start: 13 parts, among them U1 MK20LF, U3 SPI_FLASH-X25XXSMD, Y1 CRYSTAL32-SMD

Commit message: Mash up of MCHCK with TinyK20-like pinout
Parts:
- removed C10: 100n, SM0603_Capa, symbol C
- removed U3: SPI_FLASH-X25XXSMD, SparkFun-SO08, symbol SPI_FLASH-X25XXSMD
- removed Y1: CRYSTAL32-SMD, SparkFun-CRYSTAL-32KHZ-SMD, symbol CRYSTAL32-SMD
- added C13, C9: 18pF, SMD-1005, symbol C-RESCUE-mchck
- added C2: 100n, SMD-1005, symbol C-RESCUE-mchck
- added K1: CONN_MICROSD, ~, symbol CONN_microSD
- added P6: JTAG, symbol CONN_5X2
- added R4, R5: 10k, SMD-1005, symbol R-RESCUE-mchck
- added S2: USER, TACT_4x3, symbol TAC_SWITCHSMD_EVQP2
- added X1: 8MHz, ~, symbol CRYSTAL
- added Y1: 32.768kHz, ~, symbol CRYSTAL
- C1, C3, C4, C5, C6, C8: symbol C -> C-RESCUE-mchck
- D1: symbol LED -> LED-RESCUE-mchck
- R3: symbol R -> R-RESCUE-mchck
- S1: value TAC_SWITCHSMD_EVQP2 -> RESET
Connections:
- net labels added: A0, A1, A18, A19, A2, A3, A4, ADC0+, ADC0-, B0, B1, B16, B17, B2, B3, C0, C1, C2, C3, C4, C5, C6, C7, D0, D1, D2, D3, D4, D5, D6, D7, RST, VBAT, VRAW, VREFH, VREFL, VREG_K20
- net labels removed: +5V, FLASH_CS, FLASH_MISO, FLASH_MOSI, FLASH_SCK, PL1, PL10, PL11, PL12, PL2, PL3, PL4, PL5, PL6, PL7, PL8, PL9, PR1, PR2, PR3, PR5, PR6, PU1, PU10, PU11, PU13, PU14, PU2, PU3, PU4, PU5, PU6, PU7, PU8, PU9, SWD_CLK, SWD_DIO, VREGUSB
- wire segments 108 -> 118
- no-connect marks 1 -> 8
Other:
- note added: "Fit C9,C13 to suit crystal"
- note added: "Optional 2-8MHz\ncrystal"
- note removed: "Optional 2-8MHz\ncrystal on A18/A19"
- note removed: "Optional SPI flash IC"

Commit message: Fix up libs and footprints for Kicad v4; remove several unused libs
Parts:
- removed P6: JTAG, symbol CONN_5X2
- added P6: JTAG, RMC:Pin_Array_5x2_SMT_1.27mm_RMC, symbol CONN_02X05
- C1, C13, C2, C3, C4, C5, C6, C9: footprint SMD-1005 -> mchck:SM0603_Capa; symbol C-RESCUE-mchck -> C
- C8: footprint SM0603_Capa -> mchck:SM0603_Capa; symbol C-RESCUE-mchck -> C
- D1: footprint LED-0603 -> LEDs:LED-0603; symbol LED-RESCUE-mchck -> LED
- K1: footprint ~ -> RMC:SD_MOLEX_47579-0001-2
- R3, R4, R5: footprint SMD-1005 -> mchck:SM0603; symbol R-RESCUE-mchck -> R
- S1, S2: footprint TACT_4x3 -> RMC:SW_C&K_KMR4_ALT
- U1: footprint LQFP48 -> mchck:LQFP48
- X1: footprint ~ -> RMC:XTAL-SM-TXC-7A; symbol CRYSTAL -> Crystal
- Y1: footprint ~ -> w_crystal:crystal_tc-26_horiz; symbol CRYSTAL -> Crystal
Connections:
- net labels added: GND
- net labels removed: VSS
- wire segments 118 -> 123

Commit message: Final tidy up for V2.
Parts:
- X1: footprint RMC:XTAL-SM-TXC-7A -> Crystals:Crystal_SMD_0603_4Pads; symbol Crystal -> XTAL_TXC_7V
Connections:
- net labels removed: VREFL
- wire segments 123 -> 121
Other:
- note added: "VREFL"
Changed lines of the file:
@@
 LIBS:RMC
 LIBS:opendous
+LIBS:multireg
+LIBS:inductor_select
 LIBS:mchck-cache
 EELAYER 25 0
@@
 L C C9
 U 1 1 54C18BA2
-P 7150 5800
-F 0 "C9" H 7200 5900 50  0000 L CNN
-F 1 "18pF" H 7200 5700 50  0000 L CNN
-F 2 "mchck:SM0603_Capa" H 7150 5800 60  0001 C CNN
-F 3 "" H 7150 5800 60  0001 C CNN
-	1    7150 5800
+P 7100 5800
+F 0 "C9" H 7150 5900 50  0000 L CNN
+F 1 "18pF" H 7150 5700 50  0000 L CNN
+F 2 "mchck:SM0603_Capa" H 7100 5800 60  0001 C CNN
+F 3 "" H 7100 5800 60  0001 C CNN
+	1    7100 5800
 	1    0    0    -1
 $EndComp
@@
 $EndComp
 $Comp
-L Crystal X1
+L XTAL_TXC_7V X1
 U 1 1 54C3B144
-P 7500 5400
-F 0 "X1" H 7500 5550 60  0000 C CNN
-F 1 "8MHz" H 7500 5250 60  0000 C CNN
-F 2 "RMC:XTAL-SM-TXC-7A" H 7550 5650 60  0000 C CNN
-F 3 "~" H 7500 5400 60  0000 C CNN
-	1    7500 5400
+P 7450 5400
+F 0 "X1" H 7450 5550 60  0000 C CNN
+F 1 "8MHz" H 7450 5250 60  0000 C CNN
+F 2 "Crystals:Crystal_SMD_0603_4Pads" H 7500 5650 60  0000 C CNN
+F 3 "~" H 7450 5400 60  0000 C CNN
+	1    7450 5400
 	1    0    0    -1
 $EndComp
@@
 L R R4
 U 1 1 54C4E58A
-P 9350 3350
-F 0 "R4" V 9450 3350 50  0000 C CNN
-F 1 "10k" V 9350 3350 50  0000 C CNN
-F 2 "mchck:SM0603" H 9350 3350 60  0001 C CNN
-F 3 "" H 9350 3350 60  0001 C CNN
-	1    9350 3350
+P 9350 3250
+F 0 "R4" V 9450 3250 50  0000 C CNN
+F 1 "10k" V 9350 3250 50  0000 C CNN
+F 2 "mchck:SM0603" H 9350 3250 60  0001 C CNN
+F 3 "" H 9350 3250 60  0001 C CNN
+	1    9350 3250
 	0    -1   -1   0
 $EndComp
-NoConn ~ 9700 3450
+NoConn ~ 9700 3350
 $Comp
 L TAC_SWITCHSMD_EVQP2 S2
 U 1 1 54C4E7D4
-P 9900 3350
-F 0 "S2" H 10100 3450 50  0000 L BNN
-F 1 "USER" H 9800 3100 50  0000 L BNN
-F 2 "RMC:SW_C&K_KMR4_ALT" H 9900 3500 50  0001 C CNN
-F 3 "" H 9900 3350 60  0001 C CNN
-	1    9900 3350
+P 9900 3250
+F 0 "S2" H 10100 3350 50  0000 L BNN
+F 1 "USER" H 9800 3000 50  0000 L BNN
+F 2 "RMC:SW_C&K_KMR4_ALT" H 9900 3400 50  0001 C CNN
+F 3 "" H 9900 3250 60  0001 C CNN
+	1    9900 3250
 	1    0    0    -1
 $EndComp
@@
 Text GLabel 6050 5550 3    40   3State ~ 0
 A4
-Text GLabel 6350 5550 3    40   3State ~ 0
-A18
 Text GLabel 7650 3150 2    40   BiDi ~ 0
 C3
@@
 Text GLabel 7650 4150 2    40   3State ~ 0
 RST
-Text GLabel 7650 4250 2    40   3State ~ 0
-A19
 Text GLabel 3950 4050 0    40   Output ~ 0
 VREFH
@@
 NoConn ~ 2350 6650
 NoConn ~ 1850 6650
-Text GLabel 3750 4250 0    40   Output ~ 0
-VREFL
 Text GLabel 2750 6550 2    40   3State ~ 0
 A2
 NoConn ~ 9400 4050
-NoConn ~ 10100 3450
+NoConn ~ 10100 3350
 Text GLabel 3600 1550 2    40   3State ~ 0
 C0
@@
 	7150 4250 7650 4250
 Wire Wire Line
-	6350 5400 7350 5400
+	6350 5400 7150 5400
 Connection ~ 6350 5400
 Wire Wire Line
-	7600 5100 7600 4250
+	7600 4850 7600 4250
 Connection ~ 7600 4250
 Wire Wire Line
 	7150 3150 7650 3150
 Wire Wire Line
-	7150 3250 8950 3250
+	7150 3250 9200 3250
 Wire Wire Line
 	5350 6400 5100 6400
@@
 	2050 2700 2050 2850
 Wire Wire Line
-	7150 5950 7150 6150
-Wire Wire Line
-	7150 6150 7800 6150
+	7100 5950 7100 6150
+Wire Wire Line
+	7100 6150 7800 6150
 Wire Wire Line
 	7500 6150 7500 6300
@@
 Connection ~ 7500 6150
 Wire Wire Line
-	7800 5100 7800 5650
-Wire Wire Line
-	7150 5400 7150 5650
-Wire Wire Line
-	7600 5100 7800 5100
+	7800 4850 7800 5650
+Wire Wire Line
+	7100 5400 7100 5650
+Wire Wire Line
+	7600 4850 7800 4850
 Connection ~ 7800 5400
-Connection ~ 7150 5400
+Connection ~ 7100 5400
 Wire Wire Line
 	6050 2350 6050 1850
@@
 Wire Wire Line
 	6250 2350 6250 1850
-Connection ~ 3750 3150
 Wire Wire Line
 	5250 5150 5250 5050
@@
 	7650 3550 7150 3550
 Wire Wire Line
-	10250 3350 10250 3500
-Wire Wire Line
-	10100 3350 10250 3350
-Wire Wire Line
-	9700 3350 9500 3350
+	10250 3250 10250 3400
+Wire Wire Line
+	10100 3250 10250 3250
+Wire Wire Line
+	9700 3250 9500 3250
 Wire Wire Line
 	8300 4150 8300 4300
@@
 Wire Wire Line
 	7650 3350 7150 3350
-Wire Wire Line
-	8950 3250 8950 3350
-Wire Wire Line
-	8950 3350 9200 3350
 Text GLabel 8900 2300 0    40   3State ~ 0
 D4
@@
 L GND #PWR035
 U 1 1 566F81C6
-P 10250 3500
-F 0 "#PWR035" H 10250 3250 50  0001 C CNN
-F 1 "GND" H 10250 3350 50  0000 C CNN
-F 2 "" H 10250 3500 50  0000 C CNN
-F 3 "" H 10250 3500 50  0000 C CNN
-	1    10250 3500
+P 10250 3400
+F 0 "#PWR035" H 10250 3150 50  0001 C CNN
+F 1 "GND" H 10250 3250 50  0000 C CNN
+F 2 "" H 10250 3400 50  0000 C CNN
+F 3 "" H 10250 3400 50  0000 C CNN
+	1    10250 3400
 	1    0    0    -1
 $EndComp
@@
 	6050 6600 6050 6500
 Wire Wire Line
-	7650 5400 7800 5400
-Wire Wire Line
 	5100 6650 5250 6650
 Wire Wire Line
 	5550 6650 5700 6650
+Wire Wire Line
+	7750 5400 7800 5400
+Text Notes 3750 4250 0    40   ~ 0
+VREFL
+Text Label 6350 5550 3    40   ~ 0
+A18
+Text Label 7650 4250 2    40   ~ 0
+A19
 $EndSCHEMATC
