File: power.sch (KiCad schematic (older format))
At the start: 15 parts, among them P5 CHG, P7 LIPO, U2 MCP73831-SOT, U4 MULTIREG

Commit message: Mash up of MCHCK with TinyK20-like pinout
Parts:
- removed C2: 2.2u, SMD-1005, symbol C
- removed C7: 4.7u, SM0805, symbol CAP0805
- removed D2: CDBU0530, SOD-523F, symbol DIODE-SCHOTTKY_
- removed L1: INDUCTOR_SELECT, SM0805-3WAY, symbol INDUCTOR_SELECT
- removed P5: CHG, solderpad, symbol CONN_1
- removed P7: LIPO, SIL100-2, symbol CONN_2
- removed R4: 20k, SM0603, symbol R
- removed SJ5: SOLDERJUMPERNO, solder-jumper, symbol SOLDERJUMPERNO
- removed U2: MCP73831-SOT, SOT23-5, symbol MCP73831-SOT
- removed U4: MULTIREG, SOT23-5, symbol MULTIREG
- added U2: MCP1703_SOT23, SOT23, symbol MCP1703_SOT23
- D3: value CDBU0530 -> DIODE-SCHOTTKY_; footprint SOD-523F-NC -> (none); populate optional -> (none)
Connections:
- net labels added: VREG_K20
- net labels removed: +5V, VLIPO, VREGUSB
- wire segments 55 -> 21
Other:
- note added: "Cut track and install ferrite bead\nfor reduced analog noise\n"
- note removed: "Cut track and install ferrite beads\nfor reduced analog noise."
- note removed: "Ichg = 1000V/Rprog\nRprog = 1000V/Ichg\n\nfor 50mA, Rprog = 20k"
- note removed: "LDO, e.g. MIC5205 (16V, 150mA, 1uA Iq): bridge L/out\n\nany DC/DC regulator: bridge SJ\nstep-down, e.g. LM3671 (5.5V, 600mA, 16uA Iq): place L across L/out \nstep-up, e.g. TPS61097 (5.5V, 350mA, 5uA Iq): place L across L/in"
- note removed: "Optional LDO or DC/DC reg if 3.3V operation\nor high input voltage is required"
- note removed: "Optional LiPo charger"
- note removed: "in"
- note removed: "out"

Commit message: Fix up libs and footprints for Kicad v4; remove several unused libs
Parts:
- C11, C12: footprint SM0805 -> mchck:SM0603_Capa
- D3: footprint (none) -> mchck:SOD-523F-NC
- FB1: footprint SM0603_NC -> mchck:SM0603_NC
- SJ6: footprint SM0603_NC -> RMC:SM0603_Bridged
- U2: footprint SOT23 -> TO_SOT_Packages_SMD:SOT-23
Connections:
- net labels added: GND
- net labels removed: VSS
Changed lines of the file:
@@
 EESchema Schematic File Version 2
 LIBS:mchck-rescue
-LIBS:usb
 LIBS:power
 LIBS:device
@@
 LIBS:74xx
 LIBS:cmos4000
-LIBS:adc-dac
-LIBS:memory
-LIBS:xilinx
-LIBS:microcontrollers
-LIBS:dsp
-LIBS:microchip
-LIBS:analog_switches
-LIBS:motorola
-LIBS:texas
-LIBS:intel
-LIBS:audio
-LIBS:interface
-LIBS:digital-audio
-LIBS:philips
-LIBS:display
-LIBS:cypress
-LIBS:siliconi
-LIBS:opto
-LIBS:atmel
-LIBS:contrib
-LIBS:valves
-LIBS:microsd
-LIBS:conn_16
-LIBS:conn_15
-LIBS:conn_18
-LIBS:mcp73831
 LIBS:SparkFun
 LIBS:tac_switchsmd_evqp2
-LIBS:cn3063
-LIBS:mic5205
-LIBS:NUC120_QFN48
-LIBS:mcp1702
-LIBS:multireg
-LIBS:inductor_select
 LIBS:logo
 LIBS:MK20LF
-LIBS:mounthole
-LIBS:vssa
-LIBS:vdda
 LIBS:RMC
 LIBS:opendous
@@
 F 0 "C12" H 5000 2850 50  0000 L CNN
 F 1 "10u" H 5000 2650 50  0000 L CNN
-F 2 "SM0805" H 5000 2750 50  0001 C CNN
+F 2 "mchck:SM0603_Capa" H 5000 2750 50  0001 C CNN
 F 3 "" H 4950 2750 60  0001 C CNN
 F 4 "optional" H 4950 2750 60  0001 C CNN "populate"
@@
 F 0 "C11" H 6550 2850 50  0000 L CNN
 F 1 "10u" H 6550 2650 50  0000 L CNN
-F 2 "SM0805" H 6550 2750 50  0001 C CNN
+F 2 "mchck:SM0603_Capa" H 6550 2750 50  0001 C CNN
 F 3 "" H 6500 2750 60  0001 C CNN
 F 4 "optional" H 6500 2750 60  0001 C CNN "populate"
@@
 Wire Wire Line
 	1300 2400 2350 2400
-$Comp
-L VSS #PWR05
-U 1 1 51F00971
-P 9000 5100
-F 0 "#PWR05" H 9000 5100 30  0001 C CNN
-F 1 "VSS" H 9000 5030 30  0000 C CNN
-F 2 "" H 9000 5100 60  0001 C CNN
-F 3 "" H 9000 5100 60  0001 C CNN
-	1    9000 5100
-	1    0    0    -1
-$EndComp
 $Comp
 L FILTER FB1
@@
 F 0 "FB1" H 9450 4700 60  0000 C CNN
 F 1 "FILTER" H 9450 4450 60  0000 C CNN
-F 2 "SM0603_NC" H 9450 4550 60  0001 C CNN
+F 2 "mchck:SM0603_NC" H 9450 4550 60  0001 C CNN
 F 3 "" H 9450 4550 60  0000 C CNN
 F 4 "optional" H 9600 4700 60  0001 C CNN "populate"
@@
 	9000 4550 9100 4550
 $Comp
-L VSSA #PWR06
+L VSSA #PWR05
 U 1 1 51F00ABC
 P 9950 5100
-F 0 "#PWR06" H 9950 5100 30  0001 C CNN
+F 0 "#PWR05" H 9950 5100 30  0001 C CNN
 F 1 "VSSA" H 9950 5030 30  0000 C CNN
 F 2 "" H 9950 5100 60  0000 C CNN
@@
 $EndComp
 $Comp
-L VDDA #PWR07
+L VDDA #PWR06
 U 1 1 51F00ACB
 P 9950 4450
-F 0 "#PWR07" H 9950 4570 20  0001 C CNN
+F 0 "#PWR06" H 9950 4570 20  0001 C CNN
 F 1 "VDDA" H 9950 4540 30  0000 C CNN
 F 2 "" H 9950 4450 60  0000 C CNN
@@
 	9950 4950 9950 5100
 $Comp
-L PWR_FLAG #FLG08
+L PWR_FLAG #FLG07
 U 1 1 51F00BA3
 P 9950 4550
-F 0 "#FLG08" H 9950 4645 30  0001 C CNN
+F 0 "#FLG07" H 9950 4645 30  0001 C CNN
 F 1 "PWR_FLAG" H 9950 4730 30  0000 C CNN
 F 2 "" H 9950 4550 60  0000 C CNN
@@
 	8800 5300 8800 3950
 $Comp
-L VSS #PWR09
-U 1 1 51F1B2AE
-P 5750 3150
-F 0 "#PWR09" H 5750 3150 30  0001 C CNN
-F 1 "VSS" H 5750 3080 30  0000 C CNN
-F 2 "" H 5750 3150 60  0001 C CNN
-F 3 "" H 5750 3150 60  0001 C CNN
-	1    5750 3150
-	1    0    0    -1
-$EndComp
-$Comp
-L VDD #PWR010
+L VDD #PWR08
 U 1 1 520A18EE
 P 8100 2200
-F 0 "#PWR010" H 8100 2300 30  0001 C CNN
+F 0 "#PWR08" H 8100 2300 30  0001 C CNN
 F 1 "VDD" H 8100 2310 30  0000 C CNN
 F 2 "" H 8100 2200 60  0000 C CNN
@@
 F 0 "SJ6" H 8500 2450 50  0000 L BNN
 F 1 "SOLDERJUMPERNC" H 8600 2400 50  0001 L BNN
-F 2 "SM0603_NC" H 8600 2550 50  0001 C CNN
+F 2 "RMC:SM0603_Bridged" H 8600 2550 50  0001 C CNN
 F 3 "" H 8600 2400 60  0001 C CNN
 F 4 "never" H 8600 2400 60  0001 C CNN "populate"
@@
 $EndComp
 $Comp
-L VDD #PWR011
+L VDD #PWR09
 U 1 1 520A432C
 P 9000 4450
-F 0 "#PWR011" H 9000 4550 30  0001 C CNN
+F 0 "#PWR09" H 9000 4550 30  0001 C CNN
 F 1 "VDD" H 9000 4560 30  0000 C CNN
 F 2 "" H 9000 4450 60  0000 C CNN
@@
 $EndComp
 $Comp
-L PWR_FLAG #FLG012
+L PWR_FLAG #FLG010
 U 1 1 530CC158
 P 1600 2200
-F 0 "#FLG012" H 1600 2295 30  0001 C CNN
+F 0 "#FLG010" H 1600 2295 30  0001 C CNN
 F 1 "PWR_FLAG" H 1600 2380 30  0000 C CNN
 F 2 "" H 1600 2200 60  0000 C CNN
@@
 Connection ~ 1600 2400
 $Comp
-L VSS #PWR013
-U 1 1 530CC49B
-P 950 1850
-F 0 "#PWR013" H 950 1850 30  0001 C CNN
-F 1 "VSS" H 950 1780 30  0000 C CNN
-F 2 "" H 950 1850 60  0001 C CNN
-F 3 "" H 950 1850 60  0001 C CNN
-	1    950  1850
-	1    0    0    -1
-$EndComp
-$Comp
-L PWR_FLAG #FLG014
+L PWR_FLAG #FLG011
 U 1 1 530CC4A1
 P 950 1750
-F 0 "#FLG014" H 950 1845 30  0001 C CNN
+F 0 "#FLG011" H 950 1845 30  0001 C CNN
 F 1 "PWR_FLAG" H 950 1930 30  0000 C CNN
 F 2 "" H 950 1750 60  0000 C CNN
@@
 F 0 "U2" H 5500 2100 60  0000 C CNN
 F 1 "MCP1703_SOT23" H 5750 2550 60  0000 C CNN
-F 2 "SOT23" H 5900 2150 60  0000 C CNN
+F 2 "TO_SOT_Packages_SMD:SOT-23" H 5900 2150 60  0000 C CNN
 F 3 "~" H 5750 2400 60  0000 C CNN
 	1    5750 2400
@@
 F 0 "D3" H 2550 2419 50  0000 L BNN
 F 1 "DIODE-SCHOTTKY_" H 2550 2309 50  0000 L BNN
-F 2 "" H 2450 2550 50  0001 C CNN
+F 2 "mchck:SOD-523F-NC" H 2450 2550 50  0001 C CNN
 F 3 "" H 2450 2400 60  0000 C CNN
 	1    2450 2400
@@
 Wire Wire Line
 	9000 4950 9950 4950
+$Comp
+L GND #PWR012
+U 1 1 566F8A18
+P 9000 5100
+F 0 "#PWR012" H 9000 4850 50  0001 C CNN
+F 1 "GND" H 9000 4950 50  0000 C CNN
+F 2 "" H 9000 5100 50  0000 C CNN
+F 3 "" H 9000 5100 50  0000 C CNN
+	1    9000 5100
+	1    0    0    -1
+$EndComp
+$Comp
+L GND #PWR013
+U 1 1 566F8ADE
+P 5750 3150
+F 0 "#PWR013" H 5750 2900 50  0001 C CNN
+F 1 "GND" H 5750 3000 50  0000 C CNN
+F 2 "" H 5750 3150 50  0000 C CNN
+F 3 "" H 5750 3150 50  0000 C CNN
+	1    5750 3150
+	1    0    0    -1
+$EndComp
+$Comp
+L GND #PWR014
+U 1 1 566F8B1E
+P 950 1850
+F 0 "#PWR014" H 950 1600 50  0001 C CNN
+F 1 "GND" H 950 1700 50  0000 C CNN
+F 2 "" H 950 1850 50  0000 C CNN
+F 3 "" H 950 1850 50  0000 C CNN
+	1    950  1850
+	1    0    0    -1
+$EndComp
 $EndSCHEMATC

Commit message: Final tidy up for V2.
Connections:
- wire segments 21 -> 22
Other:
- note added: "Cut jumper if U2 fitted"
Changed lines of the file:
@@
 LIBS:RMC
 LIBS:opendous
+LIBS:multireg
+LIBS:inductor_select
 LIBS:mchck-cache
 EELAYER 25 0
@@
 L PWR_FLAG #FLG04
 U 1 1 4F25B2E7
-P 4650 2400
-F 0 "#FLG04" H 4650 2495 30  0001 C CNN
-F 1 "PWR_FLAG" H 4650 2580 30  0000 C CNN
-F 2 "" H 4650 2400 60  0001 C CNN
-F 3 "" H 4650 2400 60  0001 C CNN
-	1    4650 2400
-	1    0    0    -1
-$EndComp
-Text Notes 2050 2100 0    40   ~ 0
+P 3550 1650
+F 0 "#FLG04" H 3550 1745 30  0001 C CNN
+F 1 "PWR_FLAG" H 3550 1830 30  0000 C CNN
+F 2 "" H 3550 1650 60  0001 C CNN
+F 3 "" H 3550 1650 60  0001 C CNN
+	1    3550 1650
+	1    0    0    -1
+$EndComp
+Text Notes 2100 2200 0    40   ~ 0
 Cut track and install if VRAW\nand VBUS operation desired
 $Comp
@@
 	1    0    0    -1
 $EndComp
-Wire Notes Line
-	3000 1950 1950 1950
-Wire Notes Line
-	3000 1950 3000 2500
-Wire Notes Line
-	3000 2500 1950 2500
-Wire Notes Line
-	1950 2500 1950 1950
-Wire Wire Line
-	4950 2400 4950 2550
-Wire Wire Line
-	5750 2800 5750 3150
-Connection ~ 4950 2400
-Wire Wire Line
-	6500 2400 6500 2550
-Connection ~ 6500 2400
-Wire Notes Line
-	7000 1150 7000 3350
-Wire Notes Line
-	7000 3350 4450 3350
-Wire Notes Line
-	4450 3350 4450 1150
-Wire Notes Line
-	4450 1150 7000 1150
-Wire Wire Line
-	8100 2400 8100 2200
-Wire Wire Line
-	3550 1650 3550 2400
-Connection ~ 4650 2400
-Wire Wire Line
-	2550 2400 5350 2400
-Connection ~ 3550 2400
-Wire Wire Line
-	1300 2400 2350 2400
 $Comp
 L FILTER FB1
 U 1 1 51F00979
-P 9450 4550
-F 0 "FB1" H 9450 4700 60  0000 C CNN
-F 1 "FILTER" H 9450 4450 60  0000 C CNN
-F 2 "mchck:SM0603_NC" H 9450 4550 60  0001 C CNN
-F 3 "" H 9450 4550 60  0000 C CNN
-F 4 "optional" H 9600 4700 60  0001 C CNN "populate"
-	1    9450 4550
-	1    0    0    -1
-$EndComp
-Wire Wire Line
-	9000 5100 9000 4950
-Wire Wire Line
-	9000 4450 9000 4550
-Wire Wire Line
-	9000 4550 9100 4550
+P 8800 4500
+F 0 "FB1" H 8800 4650 60  0000 C CNN
+F 1 "FILTER" H 8800 4400 60  0000 C CNN
+F 2 "mchck:SM0603_NC" H 8800 4500 60  0001 C CNN
+F 3 "" H 8800 4500 60  0000 C CNN
+F 4 "optional" H 8950 4650 60  0001 C CNN "populate"
+	1    8800 4500
+	1    0    0    -1
+$EndComp
 $Comp
 L VSSA #PWR05
 U 1 1 51F00ABC
-P 9950 5100
-F 0 "#PWR05" H 9950 5100 30  0001 C CNN
-F 1 "VSSA" H 9950 5030 30  0000 C CNN
-F 2 "" H 9950 5100 60  0000 C CNN
-F 3 "" H 9950 5100 60  0000 C CNN
-	1    9950 5100
+P 9300 5050
+F 0 "#PWR05" H 9300 5050 30  0001 C CNN
+F 1 "VSSA" H 9300 4980 30  0000 C CNN
+F 2 "" H 9300 5050 60  0000 C CNN
+F 3 "" H 9300 5050 60  0000 C CNN
+	1    9300 5050
 	1    0    0    -1
 $EndComp
@@
 L VDDA #PWR06
 U 1 1 51F00ACB
-P 9950 4450
-F 0 "#PWR06" H 9950 4570 20  0001 C CNN
-F 1 "VDDA" H 9950 4540 30  0000 C CNN
-F 2 "" H 9950 4450 60  0000 C CNN
-F 3 "" H 9950 4450 60  0000 C CNN
-	1    9950 4450
-	1    0    0    -1
-$EndComp
-Wire Wire Line
-	9800 4550 9950 4550
-Wire Wire Line
-	9950 4550 9950 4450
-Wire Wire Line
-	9950 4950 9950 5100
+P 9300 4400
+F 0 "#PWR06" H 9300 4520 20  0001 C CNN
+F 1 "VDDA" H 9300 4490 30  0000 C CNN
+F 2 "" H 9300 4400 60  0000 C CNN
+F 3 "" H 9300 4400 60  0000 C CNN
+	1    9300 4400
+	1    0    0    -1
+$EndComp
 $Comp
 L PWR_FLAG #FLG07
 U 1 1 51F00BA3
-P 9950 4550
-F 0 "#FLG07" H 9950 4645 30  0001 C CNN
-F 1 "PWR_FLAG" H 9950 4730 30  0000 C CNN
-F 2 "" H 9950 4550 60  0000 C CNN
-F 3 "" H 9950 4550 60  0000 C CNN
-	1    9950 4550
+P 9300 4500
+F 0 "#FLG07" H 9300 4595 30  0001 C CNN
+F 1 "PWR_FLAG" H 9300 4680 30  0000 C CNN
+F 2 "" H 9300 4500 60  0000 C CNN
+F 3 "" H 9300 4500 60  0000 C CNN
+	1    9300 4500
 	0    1    1    0
 $EndComp
-Wire Notes Line
-	8800 3950 10300 3950
-Wire Notes Line
-	10300 3950 10300 5300
-Wire Notes Line
-	10300 5300 8800 5300
-Wire Notes Line
-	8800 5300 8800 3950
 $Comp
 L VDD #PWR08
 U 1 1 520A18EE
-P 8100 2200
-F 0 "#PWR08" H 8100 2300 30  0001 C CNN
-F 1 "VDD" H 8100 2310 30  0000 C CNN
-F 2 "" H 8100 2200 60  0000 C CNN
-F 3 "" H 8100 2200 60  0000 C CNN
-	1    8100 2200
+P 7050 1650
+F 0 "#PWR08" H 7050 1750 30  0001 C CNN
+F 1 "VDD" H 7050 1760 30  0000 C CNN
+F 2 "" H 7050 1650 60  0000 C CNN
+F 3 "" H 7050 1650 60  0000 C CNN
+	1    7050 1650
 	1    0    0    -1
 $EndComp
@@
 L SOLDERJUMPERNC SJ6
 U 1 1 520A195F
-P 8600 2400
-F 0 "SJ6" H 8500 2450 50  0000 L BNN
-F 1 "SOLDERJUMPERNC" H 8600 2400 50  0001 L BNN
-F 2 "RMC:SM0603_Bridged" H 8600 2550 50  0001 C CNN
-F 3 "" H 8600 2400 60  0001 C CNN
-F 4 "never" H 8600 2400 60  0001 C CNN "populate"
-	1    8600 2400
+P 7700 2400
+F 0 "SJ6" H 7700 2250 50  0000 C BNN
+F 1 "SOLDERJUMPERNC" H 7700 2400 50  0001 L BNN
+F 2 "RMC:SM0603_Bridged" H 7700 2550 50  0001 C CNN
+F 3 "" H 7700 2400 60  0001 C CNN
+F 4 "never" H 7700 2400 60  0001 C CNN "populate"
+	1    7700 2400
 	-1   0    0    1
 $EndComp
@@
 L VDD #PWR09
 U 1 1 520A432C
-P 9000 4450
-F 0 "#PWR09" H 9000 4550 30  0001 C CNN
-F 1 "VDD" H 9000 4560 30  0000 C CNN
-F 2 "" H 9000 4450 60  0000 C CNN
-F 3 "" H 9000 4450 60  0000 C CNN
-	1    9000 4450
+P 8350 4400
+F 0 "#PWR09" H 8350 4500 30  0001 C CNN
+F 1 "VDD" H 8350 4510 30  0000 C CNN
+F 2 "" H 8350 4400 60  0000 C CNN
+F 3 "" H 8350 4400 60  0000 C CNN
+	1    8350 4400
 	1    0    0    -1
 $EndComp
@@
 L PWR_FLAG #FLG010
 U 1 1 530CC158
-P 1600 2200
-F 0 "#FLG010" H 1600 2295 30  0001 C CNN
-F 1 "PWR_FLAG" H 1600 2380 30  0000 C CNN
-F 2 "" H 1600 2200 60  0000 C CNN
-F 3 "" H 1600 2200 60  0000 C CNN
-	1    1600 2200
-	1    0    0    -1
-$EndComp
-Wire Wire Line
-	1600 2200 1600 2400
-Connection ~ 1600 2400
+P 1600 2350
+F 0 "#FLG010" H 1600 2445 30  0001 C CNN
+F 1 "PWR_FLAG" H 1600 2530 30  0000 C CNN
+F 2 "" H 1600 2350 60  0000 C CNN
+F 3 "" H 1600 2350 60  0000 C CNN
+	1    1600 2350
+	1    0    0    -1
+$EndComp
 $Comp
 L PWR_FLAG #FLG011
 U 1 1 530CC4A1
-P 950 1750
-F 0 "#FLG011" H 950 1845 30  0001 C CNN
-F 1 "PWR_FLAG" H 950 1930 30  0000 C CNN
-F 2 "" H 950 1750 60  0000 C CNN
-F 3 "" H 950 1750 60  0000 C CNN
-	1    950  1750
-	1    0    0    -1
-$EndComp
-Wire Wire Line
-	950  1750 950  1850
-$Comp
-L MCP1703_SOT23 U2
-U 1 1 54C2F163
-P 5750 2400
-F 0 "U2" H 5500 2100 60  0000 C CNN
-F 1 "MCP1703_SOT23" H 5750 2550 60  0000 C CNN
-F 2 "TO_SOT_Packages_SMD:SOT-23" H 5900 2150 60  0000 C CNN
-F 3 "~" H 5750 2400 60  0000 C CNN
-	1    5750 2400
-	1    0    0    -1
-$EndComp
-Wire Wire Line
-	4950 2850 4950 3000
-Wire Wire Line
-	4950 3000 6500 3000
-Connection ~ 5750 3000
-Wire Wire Line
-	6500 3000 6500 2850
-Wire Wire Line
-	6150 2400 8400 2400
-Connection ~ 8100 2400
-Text Notes 9100 4050 0    40   ~ 0
+P 950 3450
+F 0 "#FLG011" H 950 3545 30  0001 C CNN
+F 1 "PWR_FLAG" H 950 3630 30  0000 C CNN
+F 2 "" H 950 3450 60  0000 C CNN
+F 3 "" H 950 3450 60  0000 C CNN
+	1    950  3450
+	1    0    0    -1
+$EndComp
+Text Notes 8400 4100 0    40   ~ 0
 Cut track and install ferrite bead\nfor reduced analog noise\n
 $Comp
@@
 Text GLabel 1300 2400 0    40   Input ~ 0
 VBUS
-Text GLabel 3350 1650 0    40   Input ~ 0
+Text GLabel 3300 1650 0    40   BiDi ~ 0
 VRAW
-Text GLabel 8800 2400 2    40   Input ~ 0
+Text GLabel 9850 2400 2    40   Input ~ 0
 VREG_K20
-Wire Wire Line
-	3550 1650 3350 1650
-Wire Wire Line
-	9000 4950 9950 4950
 $Comp
 L GND #PWR012
 U 1 1 566F8A18
-P 9000 5100
-F 0 "#PWR012" H 9000 4850 50  0001 C CNN
-F 1 "GND" H 9000 4950 50  0000 C CNN
-F 2 "" H 9000 5100 50  0000 C CNN
-F 3 "" H 9000 5100 50  0000 C CNN
-	1    9000 5100
+P 8350 5050
+F 0 "#PWR012" H 8350 4800 50  0001 C CNN
+F 1 "GND" H 8350 4900 50  0000 C CNN
+F 2 "" H 8350 5050 50  0000 C CNN
+F 3 "" H 8350 5050 50  0000 C CNN
+	1    8350 5050
 	1    0    0    -1
 $EndComp
@@
 L GND #PWR014
 U 1 1 566F8B1E
-P 950 1850
-F 0 "#PWR014" H 950 1600 50  0001 C CNN
-F 1 "GND" H 950 1700 50  0000 C CNN
-F 2 "" H 950 1850 50  0000 C CNN
-F 3 "" H 950 1850 50  0000 C CNN
-	1    950  1850
-	1    0    0    -1
-$EndComp
+P 950 3550
+F 0 "#PWR014" H 950 3300 50  0001 C CNN
+F 1 "GND" H 950 3400 50  0000 C CNN
+F 2 "" H 950 3550 50  0000 C CNN
+F 3 "" H 950 3550 50  0000 C CNN
+	1    950  3550
+	1    0    0    -1
+$EndComp
+$Comp
+L MCP1703_SOT23 U2
+U 1 1 54C2F163
+P 5750 2400
+F 0 "U2" H 5500 2100 60  0000 C CNN
+F 1 "MCP1703_SOT23" H 5750 2550 60  0000 C CNN
+F 2 "TO_SOT_Packages_SMD:SOT-23" H 5750 2700 60  0000 C CNN
+F 3 "~" H 5750 2400 60  0000 C CNN
+	1    5750 2400
+	1    0    0    -1
+$EndComp
+Wire Wire Line
+	4950 2400 4950 2550
+Wire Wire Line
+	5750 2800 5750 3150
+Connection ~ 4950 2400
+Wire Wire Line
+	6500 2400 6500 2550
+Connection ~ 6500 2400
+Wire Notes Line
+	8350 3350 8350 1150
+Wire Notes Line
+	4450 3350 8350 3350
+Wire Notes Line
+	4450 3350 4450 1150
+Wire Notes Line
+	4450 1150 8350 1150
+Wire Wire Line
+	7050 2400 7050 1650
+Wire Wire Line
+	3550 1650 3550 2400
+Wire Wire Line
+	2550 2400 5350 2400
+Connection ~ 3550 2400
+Wire Wire Line
+	1300 2400 2350 2400
+Wire Wire Line
+	8350 5050 8350 4900
+Wire Wire Line
+	8350 4400 8350 4500
+Wire Wire Line
+	8350 4500 8450 4500
+Wire Wire Line
+	9150 4500 9300 4500
+Wire Wire Line
+	9300 4500 9300 4400
+Wire Wire Line
+	9300 4900 9300 5050
+Wire Notes Line
+	8150 3900 9650 3900
+Wire Notes Line
+	9650 3900 9650 5250
+Wire Notes Line
+	9650 5250 8150 5250
+Wire Notes Line
+	8150 5250 8150 3900
+Wire Wire Line
+	1600 2350 1600 2400
+Connection ~ 1600 2400
+Wire Wire Line
+	950  3450 950  3550
+Wire Wire Line
+	4950 2850 4950 3000
+Wire Wire Line
+	4950 3000 6500 3000
+Connection ~ 5750 3000
+Wire Wire Line
+	6500 3000 6500 2850
+Wire Wire Line
+	6150 2400 7500 2400
+Connection ~ 7050 2400
+Wire Wire Line
+	3550 1650 3300 1650
+Wire Wire Line
+	8350 4900 9300 4900
+Connection ~ 3550 1650
+Text Notes 7200 2150 0    60   ~ 0
+Cut jumper if U2 fitted
+Wire Wire Line
+	7900 2400 9850 2400
+Wire Notes Line
+	1950 1400 1950 2700
+Wire Notes Line
+	1950 2700 3800 2700
+Wire Notes Line
+	3800 2700 3800 1400
+Wire Notes Line
+	3800 1400 1950 1400
 $EndSCHEMATC
